File: zm31-tandymod-plus-rom-adapter.kicad_pcb (KiCad board)
At the start: 2 copper layers, 40.6 x 33 mm, 3 parts

Commit message: Update with the named nets
Parts:
- TandyMod+ ROM: value 27C512 -> ROM Socket
- ZM31: value 74LS157 -> ZM31 Socket
Connections:
- net Net-(SW1-Pad2) renamed /~TANDY
- net Net-(U1-Pad1) renamed /SEL
- net Net-(U1-Pad10) renamed /XA16
- net Net-(U1-Pad11) renamed /PG2
- net Net-(U1-Pad15) renamed /~ENABLE
- net Net-(U1-Pad2) renamed /PG0
- net Net-(U1-Pad3) renamed /XA14
- net Net-(U1-Pad4) renamed /OUT14
- net Net-(U1-Pad5) renamed /PG1
- net Net-(U1-Pad6) renamed /XA15
- net Net-(U1-Pad7) renamed /OUT15
- net Net-(U1-Pad9) renamed /OUT16
